File: CAMERA.kicad_pcb (KiCad board)
At the start: 6 copper layers, 88 parts, among them J1 Conn_01x06_Male, J10 E, J11 F, J12 G, J13 H, J14 J, J15 K, J16 L, J17 M, J18 N, J19 P, J2 Conn_01x08_Male, J20 R, J21 T, J22 Conn_01x10_Male, J23 Conn_01x08_Male, J26 Conn_01x25_Pin, J27 Conn_01x25_Pin, J28 Conn_01x25_Pin, J29 Conn_01x25_Pin, J3 A, J4 U, J5 B, J6 V, J7 C, J8 W, J9 D, Q1 BC550

Commit message: Add files via upload
Parts:
- moved C3 7.92 mm to (36.4, 37.1)
- moved C13 7.62 mm to (33.0, 48.2)
- moved C4 5.15 mm to (36.2, 30.6)
- moved C21 3.62 mm to (27.9, 63.5)
- moved C22 3.54 mm to (43.2, 86.4)
- moved C17 2.58 mm to (43.2, 35.6)
- moved C5 2.58 mm to (114.3, 78.7)
- moved C9 2.54 mm to (83.8, 104.1)
Routing:
- net GND: track 952.8 -> 992.5 mm, vias 3 -> 2
- net (no net): track 0.00 -> 17.2 mm
- net Net-(J17-Pin_18): track 114.3 -> 101.0 mm, vias 3 -> 2
- net Net-(J17-Pin_3): track 189.0 -> 181.9 mm
- net +3.3V: track 925.1 -> 918.5 mm
- net DATA39: track 145.1 -> 139.4 mm
- net Net-(J14-Pin_17): track 288.9 -> 284.5 mm
- net DATA59: track 175.3 -> 172.0 mm
- net DATA36: track 138.0 -> 135.8 mm
- net DATA38: track 69.8 -> 67.7 mm
- net DATA87: track 319.2 -> 321.0 mm
- net DATA14: track 61.6 -> 60.3 mm
- net DATA37: track 149.6 -> 148.4 mm
- net DATA91: track 278.8 -> 278.1 mm
- net DATA21: track 90.0 -> 89.3 mm
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Other:
- board text added: "Picot en bas à gauche en vue de dessus Gestion d'un capteur d'image MT9M413 Version 2, 12/04/2025, Edern Ollivier"
- board text removed: "Picot en bas à gauche en vue de dessus Gestion d'un capteur d'image MT9M413 Version 2, 21/05/2025, Edern Ollivier"

Commit message: Add files via upload
Routing:
- net Net-(J10-Pin_18): track 214.3 -> 228.6 mm
- net Net-(J17-Pin_3): track 181.9 -> 173.1 mm, vias 0 -> 2
- net Net-(J12-Pin_15): track 186.9 -> 187.8 mm
Changed lines of the file:
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@@
 	)
 	(segment
+		(start 248.873959 83.773959)
+		(end 238.76 73.66)
+		(width 0.25)
+		(layer "F.Cu")
+		(net 135)
+	)
+	(segment
 		(start 246.115 85.655)
 		(end 247.29 86.83)
@@
 	)
 	(segment
+		(start 241.035 86.095)
+		(end 241.266095 86.326095)
+		(width 0.25)
+		(layer "F.Cu")
+		(net 144)
+	)
+	(segment
 		(start 75.024 66.04)
 		(end 75.024 65.552884)
@@
 	)
 	(segment
+		(start 243.75 86.141701)
+		(end 243.75 85.168299)
+		(width 0.25)
+		(layer "F.Cu")
+		(net 161)
+	)
+	(segment
 		(start 229.071 86.831)
 		(end 223.619 86.831)
@@
 	(segment
 		(start 237.131 86.142116)
-		(end 237.131 79.651)
+		(end 237.131 85.167884)
 		(width 0.25)
 		(layer "B.Cu")
@@
 	)
 	(segment
+		(start 237.131 85.167884)
+		(end 237.131 79.651)
+		(width 0.25)
+		(layer "B.Cu")
+		(net 169)
+	)
+	(segment
 		(start 225.5 78.74)
 		(end 232.248611 78.74)
@@
 	)
 	(segment
-		(start 86.526 27.774)
-		(end 80.104 34.196)
+		(start 83.333299 51.975)
+		(end 82.455 51.096701)
 		(width 0.25)
-		(layer "In3.Cu")
+		(layer "F.Cu")
 		(net 245)
 	)
 	(segment
-		(start 129.374 27.774)
-		(end 86.526 27.774)
+		(start 77.565 47.773299)
+		(end 76.686701 46.895)
 		(width 0.25)
-		(layer "In3.Cu")
+		(layer "F.Cu")
 		(net 245)
 	)
 	(segment
-		(start 129.54 27.94)
-		(end 129.374 27.774)
+		(start 75.579177 46.760878)
+		(end 75.190505 46.760878)
 		(width 0.25)
-		(layer "In3.Cu")
+		(layer "F.Cu")
 		(net 245)
 	)
 	(segment
-		(start 80.104 41.816)
-		(end 78.74 43.18)
+		(start 77.565 48.746701)
+		(end 77.565 47.773299)
 		(width 0.25)
-		(layer "In3.Cu")
+		(layer "F.Cu")
 		(net 245)
 	)
 	(segment
-		(start 225.795 85.655)
-		(end 168.08 27.94)
+		(start 82.455 49.935)
+		(end 81.955 49.435)
 		(width 0.25)
-		(layer "In3.Cu")
+		(layer "F.Cu")
 		(net 245)
 	)
 	(segment
-		(start 80.104 34.196)
-		(end 80.104 41.816)
+		(start 78.253299 49.435)
+		(end 77.565 48.746701)
 		(width 0.25)
-		(layer "In3.Cu")
+		(layer "F.Cu")
 		(net 245)
 	)
 	(segment
-		(start 168.08 27.94)
-		(end 129.54 27.94)
+		(start 99.995 51.975)
+		(end 83.333299 51.975)
 		(width 0.25)
-		(layer "In3.Cu")
+		(layer "F.Cu")
+		(net 245)
+	)
+	(segment
+		(start 101.735 53.715)
+		(end 99.995 51.975)
+		(width 0.25)
+		(layer "F.Cu")
+		(net 245)
+	)
+	(segment
+		(start 75.713299 46.895)
+		(end 75.579177 46.760878)
+		(width 0.25)
+		(layer "F.Cu")
+		(net 245)
+	)
+	(segment
+		(start 81.955 49.435)
+		(end 78.253299 49.435)
+		(width 0.25)
+		(layer "F.Cu")
+		(net 245)
+	)
+	(segment
+		(start 76.686701 46.895)
+		(end 75.713299 46.895)
+		(width 0.25)
+		(layer "F.Cu")
+		(net 245)
+	)
+	(segment
+		(start 82.455 51.096701)
+		(end 82.455 49.935)
+		(width 0.25)
+		(layer "F.Cu")
+		(net 245)
+	)
+	(via
+		(at 101.735 53.715)
+		(size 0.8)
+		(drill 0.4)
+		(layers "F.Cu" "B.Cu")
+		(net 245)
+	)
+	(via
+		(at 75.190505 46.760878)
+		(size 0.8)
+		(drill 0.4)
+		(layers "F.Cu" "B.Cu")
+		(net 245)
+	)
+	(segment
+		(start 77.375 44.545)
+		(end 75.735 44.545)
+		(width 0.25)
+		(layer "B.Cu")
+		(net 245)
+	)
+	(segment
+		(start 75.025 45.233299)
+		(end 75.639149 44.61915)
+		(width 0.25)
+		(layer "B.Cu")
+		(net 245)
+	)
+	(segment
+		(start 224.795 85.655)
+		(end 133.675 85.655)
+		(width 0.25)
+		(layer "B.Cu")
+		(net 245)
+	)
+	(segment
+		(start 75.66085 44.61915)
+		(end 75.735 44.545)
+		(width 0.25)
+		(layer "B.Cu")
+		(net 245)
+	)
+	(segment
+		(start 78.74 43.18)
+		(end 77.375 44.545)
+		(width 0.25)
+		(layer "B.Cu")
+		(net 245)
+	)
+	(segment
+		(start 75.190505 46.760878)
+		(end 75.025 46.595373)
+		(width 0.25)
+		(layer "B.Cu")
+		(net 245)
+	)
+	(segment
+		(start 75.025 46.595373)
+		(end 75.025 45.233299)
+		(width 0.25)
+		(layer "B.Cu")
+		(net 245)
+	)
+	(segment
+		(start 75.639149 44.61915)
+		(end 75.66085 44.61915)
+		(width 0.25)
+		(layer "B.Cu")
+		(net 245)
+	)
+	(segment
+		(start 133.675 85.655)
+		(end 101.735 53.715)
+		(width 0.25)
+		(layer "B.Cu")
 		(net 245)
 	)
@@
 		(width 0.25)
 		(layer "B.Cu")
+		(net 308)
+	)
+	(segment
+		(start 228.335 86.095)
+		(end 228.6 86.36)
+		(width 0.25)
+		(layer "B.Cu")

Commit message: Add files via upload
Parts:
- moved C3 11.7 mm to (36.1, 25.4)
- moved C4 10.7 mm to (33.0, 20.3)
- moved C13 7.62 mm to (25.4, 48.2)
- moved C5 5.12 mm to (119.4, 78.7)
- moved C6 5.12 mm to (119.4, 86.4)
- moved C19 5.08 mm to (91.4, 109.2)
- moved C22 5.08 mm to (48.3, 86.4)
- moved C9 5.08 mm to (83.8, 109.2)
- moved C12 3.62 mm to (25.4, 81.3)
- moved C21 3.62 mm to (25.4, 66.1)
- moved C17 2.58 mm to (45.8, 35.6)
- moved C8 2.54 mm to (104.1, 101.6)
Routing:
- net +3.3V: track 918.5 -> 987.1 mm, vias 2 -> 4
- net GND: track 992.5 -> 1060.5 mm, vias 2 -> 5
- net (no net): track 17.2 -> 0.00 mm
- net Net-(J11-Pin_16): track 264.8 -> 249.6 mm
- net Net-(J10-Pin_18): track 228.6 -> 214.3 mm
- net Net-(J17-Pin_18): track 101.0 -> 112.3 mm
- net DATA59: track 172.0 -> 182.7 mm
- net Net-(J17-Pin_3): track 173.1 -> 181.9 mm, vias 2 -> 0
- net Net-(J16-Pin_15): track 363.1 -> 367.6 mm
- net DATA39: track 139.4 -> 135.0 mm
- net Net-(J14-Pin_17): track 284.5 -> 288.9 mm
- net DATA36: track 135.8 -> 139.8 mm
- net DATA87: track 321.0 -> 325.0 mm
- net DATA61: track 104.0 -> 107.5 mm
- net DATA60: track 104.4 -> 107.7 mm
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Other:
- board text added: "Picot en bas à gauche en vue de dessus Gestion d'un capteur d'image MT9M413 Version 2, 10/06/2025, Edern Ollivier"
- board text removed: "Picot en bas à gauche en vue de dessus Gestion d'un capteur d'image MT9M413 Version 2, 12/04/2025, Edern Ollivier"

Commit message: Add files via upload
Parts:
- moved C14 18.6 mm to (75.0, 104.9)
- moved C18 18.6 mm to (57.2, 104.9)
- moved C20 18.6 mm to (92.8, 104.9)
- moved C22 18.4 mm to (50.2, 104.6)
- moved C7 18.3 mm to (47.0, 119.9)
- moved C10 17.9 mm to (55.8, 48.4)
- moved JP1 17.8 mm to (211.5, 77.9)
- moved ? 17.8 mm to (120.7, 48.4)
- moved ? 17.8 mm to (120.7, 109.2)
- moved C19 17.8 mm to (92.8, 127.0)
- moved C23 17.8 mm to (231.1, 152.4)
- moved C28 17.8 mm to (251.3, 152.4)
- moved C33 17.8 mm to (263.0, 151.3)
- moved C34 17.8 mm to (266.1, 131.7)
- moved C36 17.8 mm to (266.1, 144.8)
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Routing:
- net Net-(J17-Pin_3): track 181.9 -> 209.5 mm
- net Net-(J17-Pin_18): track 112.3 -> 117.9 mm
- net Net-(J16-Pin_16): track 312.8 -> 308.0 mm
- net Net-(J11-Pin_16): track 249.6 -> 245.5 mm
- net Net-(J12-Pin_3): track 229.2 -> 225.4 mm
- net +3.3V: track 987.1 -> 990.3 mm
- net DATA4: track 92.5 -> 94.7 mm
- net Net-(J12-Pin_18): track 214.6 -> 216.1 mm
- net Net-(J18-Pin_17): track 233.0 -> 234.4 mm
- net Net-(J14-Pin_17): track 288.9 -> 287.6 mm
- net GND: track 1060.5 -> 1061.7 mm
- net DATA99: track 290.0 -> 289.1 mm
- net DATA94: track 297.6 -> 296.6 mm
- net DATA97: track 281.4 -> 280.5 mm
- net DATA87: track 325.0 -> 325.7 mm
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Other:
- board outline added: 256.5 x 127.1 mm
- board text added: "Cercle pour visser le cache de la caméra sur la carte de gestion du capteur d'image"
